File: Page3.kicad_sch (KiCad schematic)
At the start: 28 parts

Commit message: latest rev
Parts:
- gave numbers to parts that had none: 28
Connections:
- net ETH_8 is gone; now on net GND: J601.13 (CH1)
- net ETH_9 is gone; now on net GND: J601.14 (CH2)
Other:
- moved on the sheet: C603
