File: Page1.kicad_sch (KiCad schematic)
At the start: 18 parts

Commit message: latest rev
Parts:
- gave numbers to parts that had none: 18

Commit message: V0.1 for review
Parts:
- removed C501: ${VALUE}, CAP:CAP_0603, symbol EXACT_CAP:1-00004
- removed R501: ${VALUE}, RES:RES_0603, symbol EXACT_RES:RC0603FR-072K2L
- removed R502: ${VALUE}, RES:RES_0603, symbol EXACT_RES:1-01215
- removed R503, R504, R505: ${VALUE}, RES:RES_0603, symbol EXACT_RES:RC0603FR-0747KL
- removed U501: TMP1826NGRR, IC:8-WSON_(2.5x2.5), symbol EXACT_IC:TMP1826
- renumbered C502 to C501, C503 to C502, R511 to R501, R506 to R502, R507 to R503, R508 to R504, R509 to R505, R510 to R506, R512 to R507, U502 to U501, U503 to U502
Connections:
- net RP_ANALOG_RES_SEL2: now reaches U502.9 (S3)
- net RP_ANALOG_RES_SEL0: now reaches U502.11 (S1)
- net RP_ANALOG_RES_SEL1: now reaches U502.10 (S2)
- net RP_ANALOG_SEL0 renamed RP_ANALOG_PROBE_SEL0
- net RP_ANALOG_SEL1 renamed RP_ANALOG_PROBE_SEL1
- net RP_ANALOG_SEL2 renamed RP_ANALOG_PROBE_SEL2
- net TH_AMBIENT: no longer names the net of U501.12 (Y3)
- net VCC renamed +3V3
Other:
- moved on the sheet: C501, C502, R502, R503, R504, R505, R506, U501, U502
