File: FAN-TEC-HEATER.kicad_sch (KiCad schematic)
At the start: 9 parts

Commit message: latest rev
Parts:
- gave numbers to parts that had none: 9
Changed lines of the file:
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@@
 		(on_board yes)
 		(dnp no)
-		(fields_autoplaced yes)
-		(property "Reference" "#PWR01"
+		(property "Reference" "#PWR0401"
 			(at 92.71 57.15 0)
 			(effects
@@
 		)
 		(property "Value" "VCC"
-			(at 92.71 48.26 0)
+			(at 92.456 49.784 0)
 			(effects
 				(font
@@
 			(project "etc-em3-fixture"
 				(path "/157a64f5-4f62-4631-b01d-779d24d7ed20/799e22f6-9b5e-43db-847c-48d7ef8dbb72"
-					(reference "#PWR01")
+					(reference "#PWR0401")
 					(unit 1)
 				)
@@
 		(on_board yes)
 		(dnp no)
-		(property "Reference" "#PWR03"
+		(property "Reference" "#PWR0403"
 			(at 110.49 63.5 0)
 			(effects
@@
 			(project "etc-em3-fixture"
 				(path "/157a64f5-4f62-4631-b01d-779d24d7ed20/799e22f6-9b5e-43db-847c-48d7ef8dbb72"
-					(reference "#PWR03")
+					(reference "#PWR0403")
 					(unit 1)
 				)
@@
 		(dnp no)
 		(fields_autoplaced yes)
-		(property "Reference" "K?"
+		(property "Reference" "K401"
 			(at 203.835 73.66 0)
 			(effects
@@
 			(project "etc-em3-fixture"
 				(path "/157a64f5-4f62-4631-b01d-779d24d7ed20/799e22f6-9b5e-43db-847c-48d7ef8dbb72"
-					(reference "K?")
+					(reference "K401")
 					(unit 1)
 				)
@@
 		(on_board yes)
 		(dnp no)
-		(property "Reference" "C?"
-			(at 133.35 56.134 0)
+		(property "Reference" "C402"
+			(at 135.89 53.594 0)
 			(effects
 				(font
@@
 			(project "etc-em3-fixture"
 				(path "/157a64f5-4f62-4631-b01d-779d24d7ed20/799e22f6-9b5e-43db-847c-48d7ef8dbb72"
-					(reference "C?")
+					(reference "C402")
 					(unit 1)
 				)
@@
 		(on_board yes)
 		(dnp no)
-		(property "Reference" "C?"
-			(at 98.044 54.356 0)
+		(property "Reference" "C401"
+			(at 100.076 52.578 0)
 			(effects
 				(font
@@
 			(project "etc-em3-fixture"
 				(path "/157a64f5-4f62-4631-b01d-779d24d7ed20/799e22f6-9b5e-43db-847c-48d7ef8dbb72"
-					(reference "C?")
+					(reference "C401")
 					(unit 1)
 				)
@@
 		(on_board yes)
 		(dnp no)
-		(property "Reference" "C?"
-			(at 133.35 61.214 0)
+		(property "Reference" "C403"
+			(at 135.382 65.278 0)
 			(effects
 				(font
@@
 			(project "etc-em3-fixture"
 				(path "/157a64f5-4f62-4631-b01d-779d24d7ed20/799e22f6-9b5e-43db-847c-48d7ef8dbb72"
-					(reference "C?")
+					(reference "C403")
 					(unit 1)
 				)
@@
 		(on_board yes)
 		(dnp no)
-		(property "Reference" "D?"
+		(property "Reference" "D401"
 			(at 187.96 100.838 90)
 			(effects
@@
 			(project "etc-em3-fixture"
 				(path "/157a64f5-4f62-4631-b01d-779d24d7ed20/799e22f6-9b5e-43db-847c-48d7ef8dbb72"
-					(reference "D?")
+					(reference "D401")
 					(unit 1)
 				)
@@
 		(on_board yes)
 		(dnp no)
-		(property "Reference" "#PWR05"
+		(property "Reference" "#PWR0406"
 			(at 146.05 66.04 0)
 			(effects
@@
 			(project "etc-em3-fixture"
 				(path "/157a64f5-4f62-4631-b01d-779d24d7ed20/799e22f6-9b5e-43db-847c-48d7ef8dbb72"
-					(reference "#PWR05")
+					(reference "#PWR0406")
 					(unit 1)
 				)
@@
 		(dnp no)
 		(fields_autoplaced yes)
-		(property "Reference" "J?"
+		(property "Reference" "J403"
 			(at 173.99 87.6301 0)
 			(effects
@@
 			(project "etc-em3-fixture"
 				(path "/157a64f5-4f62-4631-b01d-779d24d7ed20/799e22f6-9b5e-43db-847c-48d7ef8dbb72"
-					(reference "J?")
+					(reference "J403")
 					(unit 1)
 				)
@@
 		(on_board yes)
 		(dnp no)
-		(property "Reference" "#PWR021"
+		(property "Reference" "#PWR0407"
 			(at 185.42 101.6 0)
 			(effects
@@
 			(project "etc-em3-fixture"
 				(path "/157a64f5-4f62-4631-b01d-779d24d7ed20/799e22f6-9b5e-43db-847c-48d7ef8dbb72"
-					(reference "#PWR021")
+					(reference "#PWR0407")
 					(unit 1)
 				)
@@
 		(on_board yes)
 		(dnp no)
-		(property "Reference" "U?"
-			(at 88.646 60.706 0)
+		(property "Reference" "U401"
+			(at 88.646 58.674 0)
 			(effects
 				(font
@@
 			(project "etc-em3-fixture"
 				(path "/157a64f5-4f62-4631-b01d-779d24d7ed20/799e22f6-9b5e-43db-847c-48d7ef8dbb72"
-					(reference "U?")
+					(reference "U401")
 					(unit 1)
 				)
@@
 		(on_board yes)
 		(dnp no)
-		(property "Reference" "#PWR020"
+		(property "Reference" "#PWR0408"
 			(at 217.17 105.41 0)
 			(effects
@@
 			(project "etc-em3-fixture"
 				(path "/157a64f5-4f62-4631-b01d-779d24d7ed20/799e22f6-9b5e-43db-847c-48d7ef8dbb72"
-					(reference "#PWR020")
+					(reference "#PWR0408")
 					(unit 1)
 				)
@@
 		(on_board yes)
 		(dnp no)
-		(property "Reference" "J?"
+		(property "Reference" "J402"
 			(at 136.398 80.772 0)
 			(effects
@@
 			(project "etc-em3-fixture"
 				(path "/157a64f5-4f62-4631-b01d-779d24d7ed20/799e22f6-9b5e-43db-847c-48d7ef8dbb72"
-					(reference "J?")
+					(reference "J402")
 					(unit 1)
 				)
@@
 		(dnp no)
 		(fields_autoplaced yes)
-		(property "Reference" "#PWR023"
+		(property "Reference" "#PWR0405"
 			(at 130.81 55.88 0)
 			(effects
@@
 			(project ""
 				(path "/157a64f5-4f62-4631-b01d-779d24d7ed20/799e22f6-9b5e-43db-847c-48d7ef8dbb72"
-					(reference "#PWR023")
+					(reference "#PWR0405")
 					(unit 1)
 				)
@@
 		(dnp no)
 		(fields_autoplaced yes)
-		(property "Reference" "J?"
+		(property "Reference" "J401"
 			(at 139.7 137.1599 0)
 			(effects
@@
 			(project ""
 				(path "/157a64f5-4f62-4631-b01d-779d24d7ed20/799e22f6-9b5e-43db-847c-48d7ef8dbb72"
-					(reference "J?")
+					(reference "J401")
 					(unit 1)
 				)
@@
 		(dnp no)
 		(fields_autoplaced yes)
-		(property "Reference" "#PWR04"
+		(property "Reference" "#PWR0404"
 			(at 121.92 90.17 0)
 			(effects
@@
 			(project "etc-em3-fixture"
 				(path "/157a64f5-4f62-4631-b01d-779d24d7ed20/799e22f6-9b5e-43db-847c-48d7ef8dbb72"
-					(reference "#PWR04")
+					(reference "#PWR0404")
 					(unit 1)
 				)
@@
 		(on_board yes)
 		(dnp no)
-		(property "Reference" "#PWR02"
+		(property "Reference" "#PWR0402"
 			(at 96.52 106.68 0)
 			(effects
@@
 			(project "etc-em3-fixture"
 				(path "/157a64f5-4f62-4631-b01d-779d24d7ed20/799e22f6-9b5e-43db-847c-48d7ef8dbb72"
-					(reference "#PWR02")
+					(reference "#PWR0402")
 					(unit 1)
 				)

Commit message: V0.1 for review
Parts:
- removed D401: ${VALUE}, DIO:SOD323, symbol EXACT_DIO:1-00527
- removed K401: G2RL-2, Relay_THT:Relay_DPDT_Omron_G2RL-2, symbol Relay:G2RL-2
- added C404, C405, C406, C407, C408: ${VALUE}, CAP:CAP_0603, symbol EXACT_CAP:1-00004
- added J404: 1-01320, CONN:TE_640454-2, symbol EXACT_CONN:1-01320
- added J405: 0010321031, CONN:10-32-1031, symbol EXACT_CONN:1-00532
- added R401: ${VALUE}, RES:RES_0603, symbol EXACT_RES:1-00015
- added U402: 1-00780, IC:IC_ADS1115IRUGR, symbol EXACT_IC:1-00780
Connections:
- net GND: now also J402.2, C404.2, C405.1, C406.1, C407.1, C408.1, R401.2, U402.3 (GND)
- net PGND: no longer J402.2
- net TP34: now also J403.2
- net TP35: now also J404.1
- net TP36: now also J403.1
- net TP37: now also J404.2
- net VCC: now also C404.1, U402.8 (VDD)
- new net: C407.2, J405.2, U402.6 (AIN2)
- new net: C408.2, J405.3, U402.7 (AIN3)
- new net: C406.2, J405.1, U402.5 (AIN1)
- new net: R401.1, U402.1 (ADDR)
- new net RPI_SCL1: U402.10 (SCL)
- new net RPI_SDA1: U402.9 (SDA)
- new net SENS_TEC: C405.2, U402.4 (AIN0)
- no-connect marks 0 -> 2
Other:
- note added: "ADS1115IR"
- note added: "I2C Address 0x49"
- note added: "Voltage Test"
- moved on the sheet: C401, C402, C403, J401, J402, J403, U401

Commit message: Commit after Review
Parts:
- removed J401, J403, J404: 1-01320, CONN:TE_640454-2, symbol EXACT_CONN:1-01320
- removed J405: 0010321031, CONN:10-32-1031, symbol EXACT_CONN:1-00532
- added J101: ${MANUFACTURER PART NUMBER}, CONN:15SH-A-03-TS, symbol CONN:1-00688
- added J401, J403, J404: DME-03, CONN:B02P-VL, symbol EXACT_CONN:1-01308
Connections:
- net PGND is gone; now on net GND: C402.1, C403.2
- net +48V: now also J402.3; no longer J402.1
- net GND: now also J402.4, U401.6 (INH); no longer J402.2
- net PWM: now also J402.1; no longer J402.3
- net TACH: now also J402.2; no longer J402.4
- net TP34: now also J403.2
- net TP35: now also J404.1
- net TP36: now also J403.1
- net TP37: now also J404.2
- net TP61: no longer U401.4 (Y3)
- net TP96: now also J401.1
- net TP97: now also J401.2
- net at C407.2, U402.6 (AIN2): now also J101.2
- net at C408.2, U402.7 (AIN3): now also J101.3
- net at C406.2, U402.5 (AIN1): now also J101.1
- net TP62: no longer names the net of U401.11 (X3)
- no-connect marks 2 -> 3
Other:
- note removed: "PWM_TEC"
- note removed: "TachTEC"
- company: (none) -> Exact Technology
- title: (none) -> EM3 Fixture
