File: Peripheral test.kicad_sch (KiCad schematic)
At the start: 30 parts, among them J602 10118192-0001LF, J603 10118192-0001LF, K601 1-00784, K602 1-00784, K603 1-00784, K604 1-00784, K605 1-00784, K606 1-00784, U601 Lora1276-C1, U602 PCB Antenna 868MHz - 925MHz, U603 M95256-WMN6P

Commit message: V0.1 for review
Parts:
- gave numbers to parts that had none: 3
- renumbered C601 to C603, C602 to C604, C603 to C605
Connections:
- net L_N renamed TP22
- net TP22: no longer J603.2 (DM)
- net L_P renamed TP23
- net TP23: no longer J603.3 (DP)
- net TP40 renamed RPI_RX
- net TP41 renamed RPI_TX
- new net TP26: J603.2 (DM)
- new net TP27: J603.3 (DP)
- no-connect marks 5 -> 31
Other:
- note removed: "Ethernet"
- note removed: "RX"
- note removed: "TX"
- moved on the sheet: D601, K601

Commit message: Commit after Review
Parts:
- removed D603, D606: ${VALUE}, DIO:SOD323, symbol EXACT_DIO:1-00527
- removed J602, J603: 10118192-0001LF, CONN:101181920001LF, symbol EXACT_CONN:10118192-0001LF
- removed K603, K606: 1-00784, MISC:KEMET_UA2, symbol EXACT_MISC:1-00784
- removed R602: ${VALUE}, RES:RES_0603, symbol EXACT_RES:1-00015
- removed U603: M95256-WMN6P, Package_BGA:Texas_DSBGA-5_1.5855x1.6365mm_Layout3x2_P0.5mm, symbol Memory_EEPROM:M95256-WMN6P
- added C606: ${VALUE}, CAP:CAP_0603, symbol CAP:CC0603CRNPO9BN3R9
- added D603, D604, D605, D606, D607, D608: ESD7951ST5G, DIO:SOD923, symbol DIO:ESD7951ST5G
- added J602: 1-00084, CONN:B2B-XH-A(LF)(SN), symbol CONN:1-00084
- added J603, J604: *, CONN:MOLEX_2171820001, symbol CONN:1-01376
- added L601: ${VALUE}, IND:RES_0603, symbol IND:L-14C4N7SV4T
- added L602: ${VALUE}, IND:RES_0603, symbol IND:LQW18AS12NG0ZD
- added R601, R602, R604, R605: ${VALUE}, RES:RES_0603, symbol RES:1-00543
- added U601: M95256-WMN6P, Package_SO:SOIC-8_3.9x4.9mm_P1.27mm, symbol Memory_EEPROM:M95256-WMN6P
- renumbered C605 to C603, C603 to C604, C604 to C605, D604 to D602, D602 to D610, D605 to D612, K604 to K602, K602 to K604, K605 to K606, R601 to R603, R604 to R606, R603 to R607, R606 to R608, R605 to R609, U601 to U602, U602 to U603
Connections:
- net +3V3: now also C603.1, FB601.2, R603.1, U601.3 (~{W}), U601.7 (~{HOLD}), U601.8 (VCC)
- net GND: now also C606.1, D603.1 (A), D604.1 (A), D605.1 (A), D606.1 (A), D607.1 (A), D608.1 (A), J602.2, J603.A1 (GND), J603.A12 (GND), J603.B1 (GND), J603.B12 (GND), J603.SH1 (SHIELD), J603.SH2 (SHIELD), J603.SH3 (SHIELD), J603.SH4 (SHIELD), J604.A1 (GND), J604.A12 (GND), J604.B1 (GND), J604.B12 (GND), J604.SH1 (SHIELD), J604.SH2 (SHIELD), J604.SH3 (SHIELD), J604.SH4 (SHIELD), L601.1, R601.1, R602.1, R604.2, R605.2, U601.4 (VSS)
- net TP22: now also D604.2 (K), J604.A6 (DP1), J604.B6 (DP2)
- net TP23: now also D606.2 (K), J604.A7 (DN1), J604.B7 (DN2)
- net TP26: now also D603.2 (K), J603.A6 (DP1), J603.B6 (DP2)
- net TP27: now also D605.2 (K), J603.A7 (DN1), J603.B7 (DN2)
- net TP75: now also R608.2
- net TP77: now also R606.2
- net TP92: now also U601.2 (Q)
- net TP93: now also U601.1 (~{S})
- net TP94: now also U601.6 (C)
- net TP95: now also U601.5 (D)
- net VCC: now also J602.1; no longer C603.1, FB601.2, R603.1
- net at U602.9 (ANT): now also L601.2, L602.1
- net at U603.1 (*): now also C606.2, L602.2
- net at K601.3: now also D608.2 (K), J604.A4 (VBUS), J604.A9 (VBUS), J604.B4 (VBUS), J604.B9 (VBUS)
- net at K602.3: now also D607.2 (K), J603.A4 (VBUS), J603.A9 (VBUS), J603.B4 (VBUS), J603.B9 (VBUS)
- new net: J603.A5 (CC1), R601.2
- new net: J603.B5 (CC2), R604.1
- new net: J604.A5 (CC1), R602.2
- new net: J604.B5 (CC2), R605.1
- no-connect marks 31 -> 25
Other:
- note added: "Screen Connector"
- company: (none) -> Exact Technology
- title: (none) -> EM3 Fixture
- moved on the sheet: C601, C602, C603, C604, C605, D601, D602, D610, D612, FB601, J601, K601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
