File: POWER.kicad_sch (KiCad schematic)
At the start: 21 parts, among them J302 DME-03, U301 *, U302 1-00780

Commit message: latest rev
Parts:
- gave numbers to parts that had none: 13
- renumbered J302 to J303
Connections:
- net 3V3 renamed +3V3

Commit message: V0.1 for review
Parts:
- added C303, C306, C307, C308, C309, C316: ${VALUE}, CAP:CAP_0603, symbol EXACT_CAP:1-00004
- added C304: ${VALUE}, CAP:CAP_0603, symbol EXACT_CAP:1-01217
- added C310: ${VALUE}, CAP:CAP_1206, symbol EXACT_CAP:1-00005
- added C317: ${VALUE}, CAP:CAP_1210, symbol EXACT_CAP:1-01210
- added C318: ${VALUE}, CAP:CAP_1206, symbol EXACT_CAP:1-00029
- added R303: ${VALUE}, RES:RES_0603, symbol EXACT_RES:1-00015
- added U302: TMCS1108, IC:SOIC127P599X175-8N, symbol EXACT_IC:1-01441
- added U304: LM1085-3.3, IC:TO254P1524X483-4N, symbol EXACT_IC:1-01198
- renumbered C303 to C305, C304 to C311, C305 to C312, C306 to C313, C307 to C314, C308 to C315, R303 to R304, R304 to R305, U302 to U303
Connections:
- net PGND is gone; now on net GND: C301.2, C302.1, U301.7 (GND), U301.9 (EPAD)
- net +3V3: now also C303.1, R303.1, U302.8 (VS)
- net GND: now also C303.2, C304.1, C306.1, C307.1, C308.1, C309.1, C310.2, C316.1, C317.2, C318.1, U302.5 (GND), U304.1 (GND)
- net TP25: now also C309.2
- net TP30: now also C307.2
- net TP32: now also C308.2
- net TP33: now also C306.2
- net VCC: now also C310.1, U304.3 (VIN)
- net at J301.1: now also U302.3 (IN-), U302.4 (IN-); no longer K301.11
- new net: C316.2, C317.1, C318.2, R303.2, U304.2 (OUT), U304.4 (OUT)
- new net: K301.11, U302.1 (IN+), U302.2 (IN+)
- new net SENS_TEC: C304.2, U302.7 (VOUT)
- no-connect marks 1 -> 6
Other:
- note added: "+1V8"
- note removed: "+1V8 VDD_EXT"
- moved on the sheet: C305, C311, C312, C313, C314, C315, D301, D302, J301, J302, J303, K301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

Commit message: Commit after Review
Parts:
- added D301: ${VALUE}, DIO:SOD323, symbol EXACT_DIO:1-00527
- added D302: 1N5408, Diode_THT:D_DO-35_SOD27_P3.81mm_Vertical_KathodeUp, symbol Diode:1N5408
- added K301: G2RL-2, Relay_THT:Relay_DPDT_Omron_G2RL-2, symbol Relay:G2RL-2
- C301: footprint CAP_1K470P_PAN -> CAP:CAP_1K470P_PAN; now fitted; now in the parts list
- C302, R301: now fitted; now in the parts list
- C306, C307, C308, C309: now fitted
- C310, C316, C317, C318, R303, U304: now not fitted
- U302: renamed from U301; now fitted; now in the parts list
- renumbered D301 to D303, D302 to D304, K301 to K302, K302 to K303, U302 to U301
Connections:
- net TP25: now also C307.2, U303.5 (AIN1); no longer C309.2, U303.7 (AIN3)
- net TP30: now also C309.2, U303.7 (AIN3); no longer C307.2, U303.5 (AIN1)
- net TP32: now also C306.2, U303.4 (AIN0); no longer C308.2, U303.6 (AIN2)
- net TP33: now also C308.2, U303.6 (AIN2); no longer C306.2, U303.4 (AIN0)
- net VCC_RLY: now also D301.1 (A), K301.A2
- net at U301.3 (IN-), U301.4 (IN-): now also K302.11; no longer J301.1
- net at J301.2: now also D302.2 (A), K301.12; no longer K302.21
- net at U301.1 (IN+), U301.2 (IN+): now also J301.1; no longer K302.11
- new net: D302.1 (K), K301.11, K302.21
- new net BROWN_OUT: D301.2 (K), K301.A1
- no-connect marks 6 -> 10
Other:
- company: (none) -> Exact Technology
- title: (none) -> EM3 Fixture
- moved on the sheet: C303, C304, U301

Commit message: Review
Parts:
- added D305, D306: 1N5408, Diode_THT:D_DO-35_SOD27_P3.81mm_Vertical_KathodeUp, symbol Diode:1N5408
Connections:
- net at J301.2, K301.12: now also D305.2 (A); no longer D302.2 (A)
- net at K301.11, K302.21: now also D306.1 (K); no longer D302.1 (K)
- new net: D302.2 (A), D305.1 (K)
- new net: D302.1 (K), D306.2 (A)
Changed lines of the file:
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@@
 	)
 	(junction
-		(at 83.82 49.53)
+		(at 77.47 49.53)
 		(diameter 0)
 		(color 0 0 0 0)
@@
 		)
 	)
-	(wire
-		(pts
-			(xy 83.82 49.53) (xy 87.63 49.53)
-		)
-		(stroke
-			(width 0)
-			(type default)
-		)
-	)
 	(polyline
 		(pts
@@
 	(wire
 		(pts
+			(xy 86.36 49.53) (xy 87.63 49.53)
+		)
+		(stroke
+			(width 0)
+			(type default)
+		)
+	)
+	(wire
+		(pts
+			(xy 77.47 49.53) (xy 78.74 49.53)
+		)
+		(stroke
+			(width 0)
+			(type default)
+		)
+	)
+	(wire
+		(pts
 			(xy 252.73 129.54) (xy 252.73 127)
 		)
@@
 	(wire
 		(pts
-			(xy 83.82 45.72) (xy 83.82 49.53)
+			(xy 77.47 45.72) (xy 77.47 49.53)
 		)
 		(stroke
@@
 	(wire
 		(pts
-			(xy 49.53 49.53) (xy 83.82 49.53)
+			(xy 49.53 49.53) (xy 77.47 49.53)
 		)
 		(stroke
@@
 	(wire
 		(pts
+			(xy 77.47 45.72) (xy 83.82 45.72)
+		)
+		(stroke
+			(width 0)
+			(type default)
+		)
+	)
+	(wire
+		(pts
 			(xy 95.25 72.39) (xy 101.6 72.39)
 		)
@@
 	(wire
 		(pts
-			(xy 95.25 49.53) (xy 104.14 49.53)
+			(xy 95.25 49.53) (xy 96.52 49.53)
 		)
 		(stroke
@@
 	)
 	(symbol
+		(lib_id "Diode:1N5408")
+		(at 82.55 49.53 180)
+		(unit 1)
+		(exclude_from_sim no)
+		(in_bom yes)
+		(on_board yes)
+		(dnp no)
+		(property "Reference" "D305"
+			(at 81.534 47.244 0)
+			(effects
+				(font
+					(size 1.27 1.27)
+				)
+			)
+		)
+		(property "Value" "1N5408"
+			(at 74.93 51.054 0)
+			(effects
+				(font
+					(size 1.27 1.27)
+				)
+				(hide yes)
+			)
+		)
+		(property "Footprint" "Diode_THT:D_DO-35_SOD27_P3.81mm_Vertical_KathodeUp"
+			(at 82.55 45.085 0)
+			(effects
+				(font
+					(size 1.27 1.27)
+				)
+				(hide yes)
+			)
+		)
+		(property "Datasheet" "http://www.vishay.com/docs/88516/1n5400.pdf"
+			(at 82.55 49.53 0)
+			(effects
+				(font
+					(size 1.27 1.27)
+				)
+				(hide yes)
+			)
+		)
+		(property "Description" "1000V 3A General Purpose Rectifier Diode, DO-201AD"
+			(at 82.55 49.53 0)
+			(effects
+				(font
+					(size 1.27 1.27)
+				)
+				(hide yes)
+			)
+		)
+		(property "Sim.Device" "D"
+			(at 82.55 49.53 0)
+			(effects
+				(font
+					(size 1.27 1.27)
+				)
+				(hide yes)
+			)
+		)
+		(property "Sim.Pins" "1=K 2=A"
+			(at 82.55 49.53 0)
+			(effects
+				(font
+					(size 1.27 1.27)
+				)
+				(hide yes)
+			)
+		)
+		(pin "2"
+		)
+		(pin "1"
+		)
+		(instances
+			(project "etc-em3-fixture"
+				(path "/157a64f5-4f62-4631-b01d-779d24d7ed20/792edb8d-6e79-40ec-8a9f-e5a94d41d615"
+					(reference "D305")
+					(unit 1)
+				)
+			)
+		)
+	)
+	(symbol
 		(lib_id "power:VCC")
 		(at 242.57 72.39 0)
@@
 					(unit 1)
 				)
+			)
+		)
+	)
+	(symbol
+		(lib_id "Diode:1N5408")
+		(at 100.33 49.53 180)
+		(unit 1)
+		(exclude_from_sim no)
+		(in_bom yes)
+		(on_board yes)
+		(dnp no)
+		(property "Reference" "D306"
+			(at 99.568 47.244 0)
+			(effects
+				(font
+					(size 1.27 1.27)
+				)
+			)
+		)
+		(property "Value" "1N5408"
+			(at 92.71 51.054 0)
+			(effects
+				(font
+					(size 1.27 1.27)
+				)
+				(hide yes)
+			)
+		)
+		(property "Footprint" "Diode_THT:D_DO-35_SOD27_P3.81mm_Vertical_KathodeUp"
+			(at 100.33 45.085 0)
+			(effects
+				(font
+					(size 1.27 1.27)
+				)
+				(hide yes)
+			)
+		)
+		(property "Datasheet" "http://www.vishay.com/docs/88516/1n5400.pdf"
+			(at 100.33 49.53 0)
+			(effects
+				(font
+					(size 1.27 1.27)
+				)
+				(hide yes)
+			)
+		)
+		(property "Description" "1000V 3A General Purpose Rectifier Diode, DO-201AD"
+			(at 100.33 49.53 0)
+			(effects
+				(font
+					(size 1.27 1.27)
+				)
+				(hide yes)
+			)
+		)
+		(property "Sim.Device" "D"
+			(at 100.33 49.53 0)
+			(effects
+				(font
+					(size 1.27 1.27)
+				)
+				(hide yes)
+			)
+		)
+		(property "Sim.Pins" "1=K 2=A"
+			(at 100.33 49.53 0)
+			(effects
+				(font
+					(size 1.27 1.27)
+				)
+				(hide yes)
+			)
+		)
+		(pin "2"
+		)
+		(pin "1"
+		)
+		(instances
+			(project "etc-em3-fixture"
+				(path "/157a64f5-4f62-4631-b01d-779d24d7ed20/792edb8d-6e79-40ec-8a9f-e5a94d41d615"
+					(reference "D306")
+					(unit 1)
+				)
