File: etc-em3-fixture.kicad_pcb (KiCad board)
At the start: 2 copper layers, 101 parts, among them J301 DME-03, J302 DME-03, J303 DME-03, J401 1-01320, J402 SWR201-NRTN-S04-SA-WH, J403 1-01320, J404 1-01320, J405 0010321031, J601 SWR201-NRTN-S05-SA-WH, J602 10118192-0001LF, J603 10118192-0001LF, J701 1-00837, J702 1-00777, K301 G2RL-2, K302 G2RL-2, K601 1-00784, K602 1-00784, K603 1-00784, K604 1-00784, K605 1-00784, K606 1-00784, U301 *, U302 TMCS1108, U303 1-00780, U304 LM1085-3.3, U401 *, U402 1-00780, U501 XS3A4051PWJ, U502 XS3A4051PWJ, U601 Lora1276-C1, U602 PCB Antenna 868MHz - 925MHz, U603 M95256-WMN6P, U701 ULN2003ADRG3, U702 PCA9675PW,118, U703 ULN2003ADRG3

Commit message: Commit after Review
Parts:
- removed J405: 0010321031, CONN:10-32-1031
- removed K603: 1-00784, MISC:KEMET_UA2
- removed the K606 at (138.9, 69.5)
- removed the U603 at (173.5, 70.3)
- added C301: EEH-ZC1K470P, CAP:CAP_1K470P_PAN, F.Cu at (55.8, 50.5)
- added C606: VALUE, CAP:CAP_0603, F.Cu at (152.0, 94.2)
- added D301: VALUE, DIO:SOD323, F.Cu at (73.5, 61.2)
- added D302: 1N5408, Diode_THT:D_DO-35_SOD27_P3.81mm_Vertical_KathodeUp, F.Cu at (82.0, 36.9)
- added D604: ESD7951ST5G, DIO:SOD923, F.Cu at (163.0, 36.5)
- added D605: ESD7951ST5G, DIO:SOD923, F.Cu at (154.1, 25.0)
- added D607: ESD7951ST5G, DIO:SOD923, F.Cu at (147.9, 21.4)
- added D608: ESD7951ST5G, DIO:SOD923, F.Cu at (163.8, 39.5)
- added J101: 15SH-A-03-TS, CONN:15SH-A-03-TS, F.Cu at (131.3, 14.7)
- added J604: *, CONN:MOLEX_2171820001, F.Cu at (160.2, 37.4)
- added J703: 1-00777, CONN:TST-120-01-X-D, F.Cu at (42.7, 81.0)
- added J704: 1-00785, CONN:TSS-125-01-T-D, F.Cu at (63.9, 73.3)
- added K301: G2RL-2, Relay_THT:Relay_DPDT_Omron_G2RL-2, F.Cu at (76.9, 57.2)
- added L601: VALUE, IND:RES_0603, F.Cu at (152.0, 89.2)
- added L602: VALUE, IND:RES_0603, F.Cu at (152.8, 91.8)
- added R601: VALUE, RES:RES_0603, F.Cu at (146.8, 25.0)
- added R604: VALUE, RES:RES_0603, F.Cu at (155.9, 22.0)
- added R605: VALUE, RES:RES_0603, F.Cu at (165.0, 35.0)
- added REF**: MountingHole_3.2mm_M3, MountingHole:MountingHole_3.2mm_M3, F.Cu at (203.7, 17.1)
- added REF**: MountingHole_3.2mm_M3, MountingHole:MountingHole_3.2mm_M3, F.Cu at (23.7, 107.1)
- added REF**: MountingHole_3.2mm_M3, MountingHole:MountingHole_3.2mm_M3, F.Cu at (203.7, 107.1)
- added REF**: MountingHole_3.2mm_M3, MountingHole:MountingHole_3.2mm_M3, F.Cu at (23.6, 17.1)
- added U601: M95256-WMN6P, Package_SO:SOIC-8_3.9x4.9mm_P1.27mm, F.Cu at (62.8, 87.9)
- C302, C303, C304, C305, C306, C307, C308, C309, C310, C311, C312, C313, C314, C315, C316, C317, C318, C401, C402, C403, C404, C405, C406, C407, C408, C501, C502, C601, C602, C702, C703, D601, FB601, R301, R302, R303, R304, R305, R401, R501, R502, R503, R504, R505, R506, R507, R602, R702, R703: value ${VALUE} -> VALUE
- C603: renamed from C605; value ${VALUE} -> VALUE
- C604: renamed from C603; value ${VALUE} -> VALUE
- C605: renamed from C604; value ${VALUE} -> VALUE
- D303: renamed from D301; value ${VALUE} -> VALUE
- D304: renamed from D302; value ${VALUE} -> VALUE
- D602: renamed from D604; value ${VALUE} -> VALUE
- D603, D606: value ${VALUE} -> ESD7951ST5G; footprint DIO:SOD323 -> DIO:SOD923
- D610: renamed from D602; value ${VALUE} -> VALUE
- D612: renamed from D605; value ${VALUE} -> VALUE
- J401, J403, J404: value 1-01320 -> DME-03; footprint CONN:TE_640454-2 -> CONN:B02P-VL
- J602: value 10118192-0001LF -> 1-00084; footprint CONN:101181920001LF -> CONN:B2B-XH-A(LF)(SN)
- J603: value 10118192-0001LF -> *; footprint CONN:101181920001LF -> CONN:MOLEX_2171820001
- R603: renamed from R601; value ${VALUE} -> VALUE
- R606: renamed from R604; value ${VALUE} -> VALUE
- R607: renamed from R603; value ${VALUE} -> VALUE
- R608: renamed from R606; value ${VALUE} -> VALUE
- R609: renamed from R605; value ${VALUE} -> VALUE
- moved J403 280.3 mm to (20.2, 38.8)
- moved J404 277.9 mm to (20.2, 53.0), turned to -90 degrees
- moved J302 263.1 mm to (38.0, 25.3), turned to 0 degrees
- moved J301 210.4 mm to (80.3, 23.0), turned to 180 degrees
- moved K303 199.2 mm to (62.0, 36.6), turned to -90 degrees
- moved K302 145.8 mm to (94.2, 57.0), turned to 180 degrees
- moved J401 135.6 mm to (20.2, 68.0), turned to -90 degrees
- moved U603 126.5 mm to (152.8, 96.2), turned to -90 degrees
- moved J702 123.2 mm to (216.0, 64.4), turned to 90 degrees
- moved R603 118.4 mm to (58.0, 84.8), turned to -90 degrees
- moved C317 117.4 mm to (193.5, 103.0), turned to -90 degrees
- moved J303 115.8 mm to (177.4, 24.5), turned to 0 degrees
- moved C408 115.0 mm to (92.3, 16.2)
- moved C603 114.3 mm to (67.5, 84.8), turned to 90 degrees
- moved C407 114.0 mm to (92.3, 14.4)
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- renumbered K301 to K302, K302 to K303, K604 to K602, K602 to K604, K605 to K606, U302 to U301, U301 to U302, U601 to U602, U602 to U603
Connections:
- C306 pad 2: /Connectors/TP33 -> /Connectors/TP32
- C307 pad 2: /Connectors/TP30 -> /Connectors/TP25
- C308 pad 2: /Connectors/TP32 -> /Connectors/TP33
- C309 pad 2: /Connectors/TP25 -> /Connectors/TP30
- C402 pad 1: PGND -> GND
- C403 pad 2: PGND -> GND
- C603 pad 1: VCC -> +3V3
- D603 pad 1: VCC_RLY -> GND
- D603 pad 2: /Connectors/RLY_LED1 -> /Peripheral test/L_N
- D606 pad 1: VCC_RLY -> GND
- D606 pad 2: /Connectors/RLY_LED2 -> /Peripheral test/CPU_P
- FB601 pad 2: VCC -> +3V3
- J301 pad 2: Net-(J301-Pad2) -> Net-(D302-A)
- J402 pad 1: +48V -> /FAN-TEC-HEATER/PWM
- J402 pad 2: GND -> /FAN-TEC-HEATER/TACH
- J402 pad 3: /FAN-TEC-HEATER/PWM -> +48V
- J402 pad 4: /FAN-TEC-HEATER/TACH -> GND
- J602 pad 1: Net-(J602-VBUS) -> VCC
- J602 pad 2: /Peripheral test/CPU_N -> GND
- J702 pad 29: /Connectors/LED2 -> /Connectors/LED1
- J702 pad 31: /Connectors/LED1 -> /Connectors/LED2
- K302 pad 11: Net-(K301-Pad11) -> Net-(K302-Pad11)
- K302 pad 21: Net-(J301-Pad2) -> Net-(D302-K)
- K601 pad 3: Net-(J602-VBUS) -> Net-(D608-K)
- K602 pad 3: Net-(J603-VBUS) -> Net-(D607-K)
- R602 pad 1: Net-(U602-*) -> GND
- R602 pad 2: Net-(U601-ANT) -> Net-(J604-CC1)
- R603 pad 1: VCC -> +3V3
- R606 pad 2: Net-(K603-Pad3) -> /Connectors/TP77
- R608 pad 2: Net-(K606-Pad3) (its old number) -> /Connectors/TP75
- U301 pad 1: Net-(K301-Pad11) -> Net-(J301-Pad1)
- U301 pad 2: Net-(K301-Pad11) -> Net-(J301-Pad1)
- U301 pad 3: Net-(J301-Pad1) -> Net-(K302-Pad11)
- U301 pad 4: Net-(J301-Pad1) -> Net-(K302-Pad11)
- U303 pad 4: /Connectors/TP33 -> /Connectors/TP32
- U303 pad 5: /Connectors/TP30 -> /Connectors/TP25
- U303 pad 6: /Connectors/TP32 -> /Connectors/TP33
- U303 pad 7: /Connectors/TP25 -> /Connectors/TP30
- U401 pad 11: /Connectors/TP62 -> unconnected-(U401-X3-Pad11)
- U401 pad 4: /Connectors/TP61 -> unconnected-(U401-Y3-Pad4)
- U401 pad 6: unconnected-(U401-INH-Pad6) -> GND
- U501 pad 1: /Connectors/TP53 -> unconnected-(U501-Y4-Pad1)
- U501 pad 12: unconnected-(U501-Y3-Pad12) -> /Connectors/TP54
- U501 pad 13: unconnected-(U501-Y0-Pad13) -> /Connectors/TP50
- U501 pad 14: /Connectors/TP50 -> /Connectors/TP55
- U501 pad 15: /Connectors/TP55 -> /Connectors/TP53
- U501 pad 5: /Connectors/TP54 -> unconnected-(U501-Y5-Pad5)
- U602 pad 9: Net-(U601-ANT) -> Net-(U602-ANT)
- U701 pad 10: unconnected-(U701-7C-Pad10) -> /Connectors/RP_ANALOG_PROBE_SEL0
- U701 pad 11: /Connectors/RP_ANALOG_PROBE_SEL0 -> /Connectors/RP_ANALOG_PROBE_SEL1
- U701 pad 12: /Connectors/RP_ANALOG_PROBE_SEL1 -> /Connectors/RP_ANALOG_PROBE_SEL2
- U701 pad 13: /Connectors/RP_ANALOG_PROBE_SEL2 -> /Connectors/RP_ANALOG_RES_SEL0
- U701 pad 14: /Connectors/RP_ANALOG_RES_SEL2 -> /Connectors/RP_ANALOG_RES_SEL1
- U701 pad 15: /Connectors/RP_ANALOG_RES_SEL1 -> /Connectors/RP_ANALOG_RES_SEL2
- U701 pad 16: /Connectors/RP_ANALOG_RES_SEL0 -> /Connectors/BROWN_OUT
- U702 pad 10: Net-(U701-7B) -> Net-(U701-1B)
- U702 pad 13: /Connectors/RLY_BTN2 -> unconnected-(U702-P10-Pad13)
- U702 pad 4: Net-(U701-1B) -> Net-(U701-7B)
- U702 pad 5: Net-(U701-2B) -> Net-(U701-6B)
- U702 pad 6: Net-(U701-3B) -> Net-(U701-5B)
- U702 pad 8: Net-(U701-5B) -> Net-(U701-3B)
- U702 pad 9: Net-(U701-6B) -> Net-(U701-2B)
- U703 pad 10: /Connectors/CPU_RLY -> /Connectors/RLY_BTN2
- U703 pad 12: /Connectors/RLY_BTN1 -> /Connectors/CPU_RLY
- U703 pad 13: /Connectors/RLY_LED2 -> /Connectors/RLY_BTN1
- U703 pad 14: /Connectors/RLY_LED1 -> unconnected-(U703-3C-Pad14)
- U703 pad 15: /Connectors/VAC_RLY -> /Connectors/+48_RLY
- U703 pad 16: /Connectors/+48_RLY -> /Connectors/VAC_RLY
Routing:
- net VCC: track 0.00 -> 546.5 mm, vias 0 -> 21
- net +3V3: track 0.00 -> 475.3 mm, vias 0 -> 16
- net /Connectors/RPI_SCL1: track 0.00 -> 243.8 mm, vias 0 -> 5
- net /Connectors/RPI_SDA1: track 0.00 -> 238.2 mm, vias 0 -> 5
- net VCC_RLY: track 0.00 -> 170.2 mm, vias 0 -> 2
- net /Connectors/RP_PWM1: track 0.00 -> 168.5 mm, vias 0 -> 1
- net /Connectors/RP_PWM2: track 0.00 -> 167.5 mm, vias 0 -> 1
- net /Connectors/RESET_N: track 0.00 -> 158.6 mm, vias 0 -> 1
- net /Connectors/TP79: track 0.00 -> 156.7 mm, vias 0 -> 1
- net /Connectors/FAN_SEL2: track 0.00 -> 156.4 mm, vias 0 -> 3
- net /Connectors/FAN_SEL1: track 0.00 -> 153.5 mm, vias 0 -> 3
- net /Connectors/TP78: track 0.00 -> 150.2 mm, vias 0 -> 1
- net /Peripheral test/L_N: track 0.00 -> 128.7 mm, vias 0 -> 5
- net /Peripheral test/L_P: track 0.00 -> 128.7 mm, vias 0 -> 5
- net /Connectors/TP73: track 0.00 -> 120.3 mm, vias 0 -> 1
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- added copper zone on B.Cu, net +48V
- added copper zone on F.Cu, net +48V
- added copper zone on B.Cu, net AGND
- added copper zone on F.Cu, net AGND
- added copper zone on B.Cu, net GND
- added copper zone on F.Cu, net GND
Other:
- board outline added: 209.8 x 103 mm
- board text added: "+48VDC"
- board text added: "+48VDC IN"
- board text added: "+5VDC"
- board text added: "+5VDC IN"
- board text added: "3V3 Select"
- board text added: "AC IN"
- board text added: "Accelerometer connector"
- board text added: "Additional ADC"
- board text added: "CPU USB-C"
- board text added: "EXPANSION CONNECTOR"
- board text added: "FAN OUT"
- board text added: "FIXTURE CONN A"
- board text added: "FIXTURE CONN B"
- board text added: "GND"
- board text added: "HEATER1 OUTPUT"
- board text added: "HEATER2 OUTPUT"
- board text added: "LORA"
- board text added: "LORA ANT"
- board text added: "MODEM USB-C"
- board text added: "RPI CONN"
- board text added: "RPI Display"
- board text added: "TEC OUTPUT"

Commit message: Review
Parts:
- added D305: 1N5408, Diode_THT:D_DO-35_SOD27_P3.81mm_Vertical_KathodeUp, F.Cu at (81.4, 43.2)
- added D306: 1N5408, Diode_THT:D_DO-35_SOD27_P3.81mm_Vertical_KathodeUp, F.Cu at (81.4, 30.8)
- moved R606 3.06 mm to (126.0, 58.1)
- moved D302 0.62 mm to (81.4, 37.0)
Connections:
- J301 pad 2: Net-(D302-A) -> Net-(D305-A)
- K301 pad 11: Net-(D302-K) -> Net-(D306-K)
- K301 pad 12: Net-(D302-A) -> Net-(D305-A)
- K302 pad 21: Net-(D302-K) -> Net-(D306-K)
Routing:
- net VCC: track 546.5 -> 520.0 mm, vias 21 -> 18
- net Net-(D306-K): track 0.00 -> 17.2 mm
- net Net-(D302-K): track 9.92 -> 2.34 mm
- net /Connectors/RESET_N: track 158.6 -> 155.1 mm
- net /Peripheral test/CPU_P: track 116.9 -> 113.5 mm
- net /Connectors/LED1: track 95.9 -> 92.9 mm
- net /Peripheral test/CPU_N: track 114.2 -> 111.2 mm
- net /Connectors/TP79: track 156.7 -> 153.9 mm
- net Net-(D302-A): track 0.00 -> 2.39 mm
- net /Connectors/TP77: track 14.2 -> 12.8 mm
- net (no net): track 0.75 -> 0.00 mm
- net GND: vias 160 -> 159

Commit message: Revised PCBA
Parts:
- moved K303 22.6 mm to (50.2, 17.4), turned to 0 degrees
- moved J302 18.3 mm to (19.9, 28.4), turned to -90 degrees
- moved D304 18.0 mm to (63.0, 22.4), turned to 90 degrees
- moved J404 4.51 mm to (20.0, 57.5)
- moved J403 4.46 mm to (20.0, 43.2)
- moved J401 4.01 mm to (20.0, 72.0)
Routing:
- net GND: track 51.1 -> 109.1 mm, vias 159 -> 231
- net VCC_RLY: track 170.2 -> 206.0 mm
- net /Connectors/VAC_RLY: track 97.1 -> 122.9 mm
- net /Connectors/TP13: track 33.6 -> 56.3 mm
- net /POWER/VAC(L): track 14.2 -> 35.2 mm
- net /POWER/VAC(N): track 21.2 -> 41.5 mm
- net /Connectors/TP36: track 36.3 -> 31.8 mm
- net /Connectors/TP34: track 32.6 -> 29.1 mm
- net /Connectors/TP37: track 27.2 -> 25.3 mm
- net /Connectors/TP35: track 28.6 -> 26.9 mm
- net /Connectors/TP96: track 24.6 -> 23.1 mm
- net /Connectors/TP97: track 22.8 -> 21.6 mm
- net /Connectors/TP14: track 37.6 -> 36.9 mm
- net (no net): vias 6 -> 1
